File: atlas/atlas.kicad_sch (KiCad schematic)
At the start: 0 parts

Commit message: progress
Other:
- sheet MCU ports: added AIN0, AIN1, AIN10, AIN11, AIN12, AIN13, AIN14, AIN15, AIN2, AIN3, AIN4, AIN5, AIN6, AIN7, AIN8, AIN9, ETB1_PWM, ETB2_PWM, KNOCK_1, KNOCK_2, KNOCK_3, KNOCK_4, VR1_ANALOG, VR1_PWM, VR2_ANALOG, VR2_PWM, VR3_ANALOG, VR3_PWM, VR4_ANALOG, VR4_PWM; removed none

Commit message: hellen modules
Parts:
- added M101, M102, M103, M104: Module-vr-discrete-0.1, hellen-one-vr-discrete-0.1:vr-discrete, symbol hellen-vr:Module-vr-discrete-0.1
Connections:
- new net +5V: M101.E4 (V5_IN), M102.E4 (V5_IN), M103.E4 (V5_IN), M104.E4 (V5_IN)
- new net GND: M101.G (GND), M102.G (GND), M103.G (GND), M104.G (GND)
- new net VR_1: M101.E3 (OUT)
- new net VR_1_ANALOG: M101.E2 (OUT_A)
- new net VR_2: M102.E3 (OUT)
- new net VR_2_ANALOG: M102.E2 (OUT_A)
- new net VR_3: M103.E3 (OUT)
- new net VR_3_ANALOG: M103.E2 (OUT_A)
- new net VR_4: M104.E3 (OUT)
- new net VR_4_ANALOG: M104.E2 (OUT_A)
- new net VR_Threshold_1: M101.E1 (Thresh_IN)
- new net VR_Threshold_2: M102.E1 (Thresh_IN)
- new net VR_Threshold_3: M103.E1 (Thresh_IN)
- new net VR_Threshold_4: M104.E1 (Thresh_IN)
