File: atlas/digital_in.kicad_sch (KiCad schematic)
At the start: 72 parts

Commit message: progress
Parts:
- C401, C402, C403, C404, C405, C406, C407, C408, C409, C410, C411, C412, C413, C414, C415, C416, C417, C418, C419, C420, C421, C422, C423, C424: renamed from C?; footprint (none) -> Capacitor_SMD:C_0603_1608Metric; LCSC (none) -> C1588
- R409, R410, R411, R412, R421, R422, R423, R424, R433, R434, R435, R436: renamed from R?; footprint (none) -> Resistor_SMD:R_0603_1608Metric; LCSC (none) -> C25804
- gave numbers to parts that had none: 30
Other:
- title: (none) -> rusEFI ATLAS
