File: atlas/mcu.kicad_sch (KiCad schematic)
At the start: 31 parts, among them Y2 32khz

Commit message: progress
Parts:
- gave numbers to parts that had none: 30
- renumbered Y2 to Y302
Connections:
- net nRST: now reaches U302.34 (NRST)
Other:
- title: (none) -> rusEFI ATLAS

Commit message: pin mapping
Connections:
- net +3V3: now also C307.2, C308.2, C309.2, C310.2, C311.2, C312.2, C313.2, C314.2, C315.2, C316.2, C317.2, C318.2, C319.2, C320.2, C321.2, C322.2, C323.2, U302.103 (VDD), U302.115 (VDD), U302.124 (VDD), U302.137 (VDD33_USB), U302.15 (VDD), U302.150 (VDD), U302.158 (VDD), U302.171 (VDD), U302.185 (VDD), U302.204 (VDD), U302.26 (VDD), U302.39 (VDD), U302.52 (VDD), U302.59 (VDD), U302.73 (VDD), U302.83 (VDD), U302.94 (VDD)
- net FDCAN1_RX: now also U302.198 (PB8); no longer U302.152 (PH14)
- net FDCAN1_TX: now also U302.199 (PB9); no longer U302.151 (PH13)
- net ETB1_PWM: now reaches U302.138 (PC6)
- net ETB2_PWM: now reaches U302.139 (PC7)
- net KNOCK_1: now reaches U302.22 (PF3)
- net KNOCK_2: now reaches U302.23 (PF4)
- net KNOCK_3: now reaches U302.24 (PF5)
- net KNOCK_4: now reaches U302.27 (PF6)
- net VR1_ANALOG: now reaches U302.28 (PF7)
- net VR2_ANALOG: now reaches U302.29 (PF8)
- net VR3_ANALOG: now reaches U302.30 (PF9)
- net VR4_ANALOG: now reaches U302.31 (PF10)
- net AIN10: now reaches U302.35 (PC0)
- net AIN11: now reaches U302.36 (PC1)
- net AIN12: now reaches U302.37 (PC2_C)
- net AIN13: now reaches U302.38 (PC3_C)
- net AIN0: now reaches U302.43 (PA0)
- net AIN1: now reaches U302.44 (PA1)
- net AIN2: now reaches U302.45 (PA2)
- net AIN3: now reaches U302.50 (PA3)
- net AIN4: now reaches U302.53 (PA4)
- net AIN5: now reaches U302.54 (PA5)
- net AIN6: now reaches U302.55 (PA6)
- net AIN7: now reaches U302.56 (PA7)
- net AIN14: now reaches U302.57 (PC4)
- net AIN15: now reaches U302.58 (PC5)
- net AIN8: now reaches U302.61 (PB0)
- net AIN9: now reaches U302.62 (PB1)
- net VR1_PWM: now reaches U302.81 (PE9)
- net VR2_PWM: now reaches U302.85 (PE11)
- net VR3_PWM: now reaches U302.87 (PE13)
- net VR4_PWM: now reaches U302.88 (PE14)
Other:
- note added: "ph2-5 adc3"
Changed lines of the file:
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@@
+    (stroke (width 0) (type solid) (color 0 0 0 0))
+  )
+  (wire (pts (xy 107.315 137.16) (xy 114.3 137.16))
     (stroke (width 0) (type solid) (color 0 0 0 0))
   )
@@
     (stroke (width 0) (type solid) (color 0 0 0 0))
   )
-  (text "RTC Crystal" (at 165.1 271.145 180)
+  (polyline (pts (xy 41.275 323.85) (xy 41.275 332.74))
+    (stroke (width 0) (type dash) (color 0 0 0 0))
+  )
+  (polyline (pts (xy 41.275 332.74) (xy 49.53 332.74))
+    (stroke (width 0) (type dash) (color 0 0 0 0))
+  )
+  (polyline (pts (xy 49.53 323.85) (xy 41.275 323.85))
+    (stroke (width 0) (type dash) (color 0 0 0 0))
+  )
+  (polyline (pts (xy 49.53 323.85) (xy 49.53 332.74))
+    (stroke (width 0) (type dash) (color 0 0 0 0))
+  )
+  (text "ph2-5\nadc3" (at 48.26 329.565 180)
+    (effects (font (size 1.27 1.27)) (justify right bottom))
+  )
+  (text "RTC Crystal" (at 167.64 271.145 180)
     (effects (font (size 1.27 1.27)) (justify right bottom))
   )
@@
     )
   )
-  (hierarchical_label "FDCAN1_TX" (shape output) (at 48.895 352.425 180)
-    (effects (font (size 1.27 1.27)) (justify right))
-  )
-  (hierarchical_label "FDCAN1_RX" (shape input) (at 48.895 354.965 180)
-    (effects (font (size 1.27 1.27)) (justify right))
-  )
   (hierarchical_label "VBAT" (shape input) (at 59.055 137.16 180)
     (effects (font (size 1.27 1.27)) (justify right))
   )
+  (hierarchical_label "AIN0" (shape input) (at 125.095 146.685 0)
+    (effects (font (size 1.27 1.27)) (justify left))
+  )
+  (hierarchical_label "AIN1" (shape input) (at 125.095 149.225 0)
+    (effects (font (size 1.27 1.27)) (justify left))
+  )
+  (hierarchical_label "AIN2" (shape input) (at 125.095 151.765 0)
+    (effects (font (size 1.27 1.27)) (justify left))
+  )
+  (hierarchical_label "AIN3" (shape input) (at 125.095 154.305 0)
+    (effects (font (size 1.27 1.27)) (justify left))
+  )
+  (hierarchical_label "AIN4" (shape input) (at 125.095 156.845 0)
+    (effects (font (size 1.27 1.27)) (justify left))
+  )
+  (hierarchical_label "AIN5" (shape input) (at 125.095 159.385 0)
+    (effects (font (size 1.27 1.27)) (justify left))
+  )
+  (hierarchical_label "AIN6" (shape input) (at 125.095 161.925 0)
+    (effects (font (size 1.27 1.27)) (justify left))
+  )
+  (hierarchical_label "AIN7" (shape input) (at 125.095 164.465 0)
+    (effects (font (size 1.27 1.27)) (justify left))
+  )
+  (hierarchical_label "AIN8" (shape input) (at 125.095 189.865 0)
+    (effects (font (size 1.27 1.27)) (justify left))
+  )
+  (hierarchical_label "AIN9" (shape input) (at 125.095 192.405 0)
+    (effects (font (size 1.27 1.27)) (justify left))
+  )
   (hierarchical_label "FDCAN2_RX" (shape input) (at 125.095 202.565 0)
     (effects (font (size 1.27 1.27)) (justify left))
@@
     (effects (font (size 1.27 1.27)) (justify left))
   )
+  (hierarchical_label "FDCAN1_RX" (shape input) (at 125.095 210.185 0)
+    (effects (font (size 1.27 1.27)) (justify left))
+  )
+  (hierarchical_label "FDCAN1_TX" (shape output) (at 125.095 212.725 0)
+    (effects (font (size 1.27 1.27)) (justify left))
+  )
+  (hierarchical_label "AIN10" (shape input) (at 125.095 233.045 0)
+    (effects (font (size 1.27 1.27)) (justify left))
+  )
+  (hierarchical_label "AIN11" (shape input) (at 125.095 235.585 0)
+    (effects (font (size 1.27 1.27)) (justify left))
+  )
+  (hierarchical_label "AIN12" (shape input) (at 125.095 238.125 0)
+    (effects (font (size 1.27 1.27)) (justify left))
+  )
+  (hierarchical_label "AIN13" (shape input) (at 125.095 240.665 0)
+    (effects (font (size 1.27 1.27)) (justify left))
+  )
+  (hierarchical_label "AIN14" (shape input) (at 125.095 243.205 0)
+    (effects (font (size 1.27 1.27)) (justify left))
+  )
+  (hierarchical_label "AIN15" (shape input) (at 125.095 245.745 0)
+    (effects (font (size 1.27 1.27)) (justify left))
+  )
+  (hierarchical_label "ETB1_PWM" (shape output) (at 125.095 248.285 0)
+    (effects (font (size 1.27 1.27)) (justify left))
+  )
+  (hierarchical_label "ETB2_PWM" (shape output) (at 125.095 250.825 0)
+    (effects (font (size 1.27 1.27)) (justify left))
+  )
+  (hierarchical_label "VR1_PWM" (shape output) (at 125.095 342.265 0)
+    (effects (font (size 1.27 1.27)) (justify left))
+  )
+  (hierarchical_label "VR2_PWM" (shape output) (at 125.095 347.345 0)
+    (effects (font (size 1.27 1.27)) (justify left))
+  )
+  (hierarchical_label "VR3_PWM" (shape output) (at 125.095 352.425 0)
+    (effects (font (size 1.27 1.27)) (justify left))
+  )
+  (hierarchical_label "VR4_PWM" (shape output) (at 125.095 354.965 0)
+    (effects (font (size 1.27 1.27)) (justify left))
+  )
+  (hierarchical_label "KNOCK_1" (shape input) (at 125.095 370.205 0)
+    (effects (font (size 1.27 1.27)) (justify left))
+  )
+  (hierarchical_label "KNOCK_2" (shape input) (at 125.095 372.745 0)
+    (effects (font (size 1.27 1.27)) (justify left))
+  )
+  (hierarchical_label "KNOCK_3" (shape input) (at 125.095 375.285 0)
+    (effects (font (size 1.27 1.27)) (justify left))
+  )
+  (hierarchical_label "KNOCK_4" (shape input) (at 125.095 377.825 0)
+    (effects (font (size 1.27 1.27)) (justify left))
+  )
+  (hierarchical_label "VR1_ANALOG" (shape input) (at 125.095 380.365 0)
+    (effects (font (size 1.27 1.27)) (justify left))
+  )
+  (hierarchical_label "VR2_ANALOG" (shape input) (at 125.095 382.905 0)
+    (effects (font (size 1.27 1.27)) (justify left))
+  )
+  (hierarchical_label "VR3_ANALOG" (shape input) (at 125.095 385.445 0)
+    (effects (font (size 1.27 1.27)) (justify left))
+  )
+  (hierarchical_label "VR4_ANALOG" (shape input) (at 125.095 387.985 0)
+    (effects (font (size 1.27 1.27)) (justify left))
+  )
+  (symbol (lib_id "power:+3.3V") (at 114.3 137.16 270) (unit 1)
+    (in_bom yes) (on_board yes) (fields_autoplaced)
+    (property "Reference" "#PWR0101" (id 0) (at 110.49 137.16 0)
+      (effects (font (size 1.27 1.27)) hide)
+    )
+    (property "Value" "+3.3V" (id 1) (at 118.745 137.7949 90)
+      (effects (font (size 1.27 1.27)) (justify left))
+    )
+    (property "Footprint" "" (id 2) (at 114.3 137.16 0)
+      (effects (font (size 1.27 1.27)) hide)
+    )
+    (property "Datasheet" "" (id 3) (at 114.3 137.16 0)
+      (effects (font (size 1.27 1.27)) hide)
+    )
+    (pin "1")
+  )
   (symbol (lib_id "power:+3.3V") (at 193.04 365.125 90) (unit 1)

Commit message: progressssss
Parts:
- C326: footprint (none) -> Capacitor_SMD:C_1206_3216Metric; LCSC (none) -> C13585
Changed lines of the file:
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@@
   (symbol (lib_id "power:+3.3V") (at 114.3 137.16 270) (unit 1)
     (in_bom yes) (on_board yes) (fields_autoplaced)
-    (property "Reference" "#PWR0101" (id 0) (at 110.49 137.16 0)
+    (property "Reference" "#PWR0342" (id 0) (at 110.49 137.16 0)
       (effects (font (size 1.27 1.27)) hide)
     )
@@
   (symbol (lib_id "power:+3.3V") (at 193.04 365.125 90) (unit 1)
     (in_bom yes) (on_board yes) (fields_autoplaced)
-    (property "Reference" "#PWR0344" (id 0) (at 196.85 365.125 0)
+    (property "Reference" "#PWR0345" (id 0) (at 196.85 365.125 0)
       (effects (font (size 1.27 1.27)) hide)
     )
@@
   (symbol (lib_id "power:GND") (at 158.115 266.7 90) (unit 1)
     (in_bom yes) (on_board yes) (fields_autoplaced)
-    (property "Reference" "#PWR0342" (id 0) (at 164.465 266.7 0)
+    (property "Reference" "#PWR0343" (id 0) (at 164.465 266.7 0)
       (effects (font (size 1.27 1.27)) hide)
     )
@@
   (symbol (lib_id "power:GND") (at 158.115 273.05 90) (unit 1)
     (in_bom yes) (on_board yes) (fields_autoplaced)
-    (property "Reference" "#PWR0343" (id 0) (at 164.465 273.05 0)
+    (property "Reference" "#PWR0344" (id 0) (at 164.465 273.05 0)
       (effects (font (size 1.27 1.27)) hide)
     )
@@
   (symbol (lib_id "power:GND") (at 194.945 374.65 0) (unit 1)
     (in_bom yes) (on_board yes) (fields_autoplaced)
-    (property "Reference" "#PWR0345" (id 0) (at 194.945 381 0)
+    (property "Reference" "#PWR0346" (id 0) (at 194.945 381 0)
       (effects (font (size 1.27 1.27)) hide)
     )
@@
   (symbol (lib_id "power:GND") (at 211.455 370.205 270) (unit 1)
     (in_bom yes) (on_board yes) (fields_autoplaced)
-    (property "Reference" "#PWR0346" (id 0) (at 205.105 370.205 0)
+    (property "Reference" "#PWR0347" (id 0) (at 205.105 370.205 0)
       (effects (font (size 1.27 1.27)) hide)
     )
@@
   (symbol (lib_id "power:GND") (at 254.635 380.365 90) (unit 1)
     (in_bom yes) (on_board yes) (fields_autoplaced)
-    (property "Reference" "#PWR0347" (id 0) (at 260.985 380.365 0)
+    (property "Reference" "#PWR0348" (id 0) (at 260.985 380.365 0)
       (effects (font (size 1.27 1.27)) hide)
     )
@@
       (effects (font (size 1.27 1.27)) (justify left))
     )
-    (property "Footprint" "" (id 2) (at 195.9102 374.65 0)
+    (property "Footprint" "Capacitor_SMD:C_1206_3216Metric" (id 2) (at 195.9102 374.65 0)
       (effects (font (size 1.27 1.27)) hide)
     )
@@
       (effects (font (size 1.27 1.27)) hide)
     )
+    (property "LCSC" "C13585" (id 4) (at 194.945 370.84 0)
+      (effects (font (size 1.27 1.27)) hide)
+    )

Commit message: progress
Parts:
- added C? (x2): 100n, symbol Device:C
- added C?: 2.2u, Capacitor_SMD:C_0603_1608Metric, symbol Device:C
- added C?: C, symbol Device:C
- added FB?: FerriteBead, symbol Device:FerriteBead
- added J?: UB-20PMFP-LC7002, Connector_PinHeader_2.54mm:PinHeader_1x05_P2.54mm_Vertical, symbol Connector_Generic:Conn_01x05
- added J?: USB_B, Connector_USB:USB_B_TE_5787834_Vertical, symbol Connector:USB_B
- added J?: TC2030, Connector:Tag-Connect_TC2030-IDC-FP_2x03_P1.27mm_Vertical, symbol Connector_Generic:Conn_01x06
- added J?: FTSH-105-01-F-DV-007-K, Connector_PinHeader_1.27mm:PinHeader_2x05_P1.27mm_Vertical_SMD, symbol Connector_Generic:Conn_02x05_Odd_Even
- added R? (x2): R, symbol Device:R
- added SW?: SW_Push, symbol Switch:SW_Push
- added U?: USBLC6-2SC6, Package_TO_SOT_SMD:SOT-23-6, symbol Power_Protection:USBLC6-2SC6
Connections:
- net +3V3: now also U302.203 (PDR_ON), FB?.2, J?.1 (Pin_1), J?.1 (Pin_1), R?.1
- net GND: now also C?.1, C?.2, C?.2, C?.2, J?.3 (Pin_3), J?.4 (GND), J?.4 (Pin_4), J?.5 (Pin_5), J?.5 (Pin_5), J?.9 (Pin_9), R?.2, SW?.1, U?.2 (GND)
- net SWCLK: now also J?.4 (Pin_4), J?.4 (Pin_4)
- net SWDIO: now also J?.2 (Pin_2), J?.2 (Pin_2)
- net USB1_DM: now also J?.2 (D-), J?.2 (Pin_2), U?.3 (I/O2), U?.4 (I/O2)
- net USB1_DP: now also J?.3 (D+), J?.3 (Pin_3), U?.1 (I/O1), U?.6 (I/O1)
- net nRST: now also C?.1, J?.10 (Pin_10), J?.3 (Pin_3), R?.2, SW?.2
- net BOOT0: now reaches U302.197 (BOOT0)
- net at U302.42 (VDDA): now also C?.1, C?.2, FB?.1
- new net USB_SHIELD: C?.1, J?.5 (Pin_5), J?.5 (Shield), R?.1
- new net VBUS: J?.1 (Pin_1), J?.1 (VBUS), U?.5 (VBUS)
- no-connect marks 0 -> 4
Other:
- note added: "Cortex Debug Header"
- note added: "SD Card"
- note added: "Tag Connect TC2030"
- note added: "USB"

Commit message: hellen modules
Parts:
- gave numbers to parts that had none: 13
Changed lines of the file:
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@@
   (symbol (lib_id "power:+3.3V") (at 33.655 84.455 0) (unit 1)
     (in_bom yes) (on_board yes)
-    (property "Reference" "#PWR?" (id 0) (at 33.655 88.265 0)
+    (property "Reference" "#PWR0112" (id 0) (at 33.655 88.265 0)
       (effects (font (size 1.27 1.27)) hide)
     )
@@
   (symbol (lib_id "power:+3.3V") (at 48.895 149.225 90) (unit 1)
     (in_bom yes) (on_board yes)
-    (property "Reference" "#PWR?" (id 0) (at 52.705 149.225 0)
+    (property "Reference" "#PWR0115" (id 0) (at 52.705 149.225 0)
       (effects (font (size 1.27 1.27)) hide)
     )
@@
   (symbol (lib_id "power:+3.3V") (at 138.43 114.935 0) (unit 1)
     (in_bom yes) (on_board yes) (fields_autoplaced)
-    (property "Reference" "#PWR?" (id 0) (at 138.43 118.745 0)
+    (property "Reference" "#PWR0117" (id 0) (at 138.43 118.745 0)
       (effects (font (size 1.27 1.27)) hide)
     )
@@
   (symbol (lib_id "power:+3.3V") (at 237.49 296.545 90) (unit 1)
     (in_bom yes) (on_board yes)
-    (property "Reference" "#PWR?" (id 0) (at 241.3 296.545 0)
+    (property "Reference" "#PWR0120" (id 0) (at 241.3 296.545 0)
       (effects (font (size 1.27 1.27)) hide)
     )
@@
   (symbol (lib_id "power:+3.3V") (at 247.65 325.12 90) (unit 1)
     (in_bom yes) (on_board yes)
-    (property "Reference" "#PWR?" (id 0) (at 251.46 325.12 0)
+    (property "Reference" "#PWR0121" (id 0) (at 251.46 325.12 0)
       (effects (font (size 1.27 1.27)) hide)
     )
@@
   (symbol (lib_id "power:PWR_FLAG") (at 35.56 159.385 0) (unit 1)
     (in_bom yes) (on_board yes) (fields_autoplaced)
-    (property "Reference" "#FLG?" (id 0) (at 35.56 157.48 0)
+    (property "Reference" "#FLG0102" (id 0) (at 35.56 157.48 0)
       (effects (font (size 1.27 1.27)) hide)
     )
@@
   (symbol (lib_id "power:PWR_FLAG") (at 44.45 161.925 0) (unit 1)
     (in_bom yes) (on_board yes) (fields_autoplaced)
-    (property "Reference" "#FLG?" (id 0) (at 44.45 160.02 0)
+    (property "Reference" "#FLG0101" (id 0) (at 44.45 160.02 0)
       (effects (font (size 1.27 1.27)) hide)
     )
@@
   (symbol (lib_id "power:PWR_FLAG") (at 114.935 116.84 0) (unit 1)
     (in_bom yes) (on_board yes) (fields_autoplaced)
-    (property "Reference" "#FLG?" (id 0) (at 114.935 114.935 0)
+    (property "Reference" "#FLG0103" (id 0) (at 114.935 114.935 0)
       (effects (font (size 1.27 1.27)) hide)
     )
@@
   (symbol (lib_id "power:GND") (at 33.655 106.68 0) (unit 1)
     (in_bom yes) (on_board yes) (fields_autoplaced)
-    (property "Reference" "#PWR?" (id 0) (at 33.655 113.03 0)
+    (property "Reference" "#PWR0114" (id 0) (at 33.655 113.03 0)
       (effects (font (size 1.27 1.27)) hide)
     )
@@
   (symbol (lib_id "power:GND") (at 42.545 104.775 0) (unit 1)
     (in_bom yes) (on_board yes) (fields_autoplaced)
-    (property "Reference" "#PWR?" (id 0) (at 42.545 111.125 0)
+    (property "Reference" "#PWR0113" (id 0) (at 42.545 111.125 0)
       (effects (font (size 1.27 1.27)) hide)
     )
@@
   (symbol (lib_id "power:GND") (at 114.935 126.365 0) (unit 1)
     (in_bom yes) (on_board yes) (fields_autoplaced)
-    (property "Reference" "#PWR?" (id 0) (at 114.935 132.715 0)
+    (property "Reference" "#PWR0118" (id 0) (at 114.935 132.715 0)
       (effects (font (size 1.27 1.27)) hide)
     )
@@
   (symbol (lib_id "power:GND") (at 126.365 126.365 0) (unit 1)
     (in_bom yes) (on_board yes) (fields_autoplaced)
-    (property "Reference" "#PWR?" (id 0) (at 126.365 132.715 0)
+    (property "Reference" "#PWR0116" (id 0) (at 126.365 132.715 0)
       (effects (font (size 1.27 1.27)) hide)
     )
@@
   (symbol (lib_id "power:GND") (at 212.725 178.435 0) (unit 1)
     (in_bom yes) (on_board yes) (fields_autoplaced)
-    (property "Reference" "#PWR?" (id 0) (at 212.725 184.785 0)
+    (property "Reference" "#PWR0127" (id 0) (at 212.725 184.785 0)
       (effects (font (size 1.27 1.27)) hide)
     )
@@
   (symbol (lib_id "power:GND") (at 214.63 196.85 0) (unit 1)
     (in_bom yes) (on_board yes) (fields_autoplaced)
-    (property "Reference" "#PWR?" (id 0) (at 214.63 203.2 0)
+    (property "Reference" "#PWR0123" (id 0) (at 214.63 203.2 0)
       (effects (font (size 1.27 1.27)) hide)
     )
@@
   (symbol (lib_id "power:GND") (at 222.885 196.85 0) (unit 1)
     (in_bom yes) (on_board yes) (fields_autoplaced)
-    (property "Reference" "#PWR?" (id 0) (at 222.885 203.2 0)
+    (property "Reference" "#PWR0124" (id 0) (at 222.885 203.2 0)
       (effects (font (size 1.27 1.27)) hide)
     )
@@
   (symbol (lib_id "power:GND") (at 235.585 308.61 0) (unit 1)
     (in_bom yes) (on_board yes) (fields_autoplaced)
-    (property "Reference" "#PWR?" (id 0) (at 235.585 314.96 0)
+    (property "Reference" "#PWR0119" (id 0) (at 235.585 314.96 0)
       (effects (font (size 1.27 1.27)) hide)
     )
@@
   (symbol (lib_id "power:GND") (at 247.65 335.28 270) (unit 1)
     (in_bom yes) (on_board yes) (fields_autoplaced)
-    (property "Reference" "#PWR?" (id 0) (at 241.3 335.28 0)
+    (property "Reference" "#PWR0122" (id 0) (at 241.3 335.28 0)
       (effects (font (size 1.27 1.27)) hide)
     )
@@
   (symbol (lib_id "power:GND") (at 250.825 193.675 270) (unit 1)
     (in_bom yes) (on_board yes) (fields_autoplaced)
-    (property "Reference" "#PWR?" (id 0) (at 244.475 193.675 0)
+    (property "Reference" "#PWR0126" (id 0) (at 244.475 193.675 0)
       (effects (font (size 1.27 1.27)) hide)
     )
@@
   (symbol (lib_id "power:GND") (at 252.73 175.26 0) (unit 1)
     (in_bom yes) (on_board yes) (fields_autoplaced)
-    (property "Reference" "#PWR?" (id 0) (at 252.73 181.61 0)
+    (property "Reference" "#PWR0125" (id 0) (at 252.73 181.61 0)
       (effects (font (size 1.27 1.27)) hide)
     )
@@
   (symbol (lib_id "Device:R") (at 33.655 88.265 0) (unit 1)
     (in_bom yes) (on_board yes) (fields_autoplaced)
-    (property "Reference" "R?" (id 0) (at 35.56 87.6299 0)
+    (property "Reference" "R301" (id 0) (at 35.56 87.6299 0)
       (effects (font (size 1.27 1.27)) (justify left))
     )
@@
   (symbol (lib_id "Device:R") (at 222.885 193.04 0) (unit 1)
     (in_bom yes) (on_board yes) (fields_autoplaced)
-    (property "Reference" "R?" (id 0) (at 225.425 192.4049 0)
+    (property "Reference" "R302" (id 0) (at 225.425 192.4049 0)
       (effects (font (size 1.27 1.27)) (justify left))
     )
@@
   (symbol (lib_id "Device:C") (at 42.545 100.965 0) (unit 1)
     (in_bom yes) (on_board yes) (fields_autoplaced)
-    (property "Reference" "C?" (id 0) (at 46.355 100.3299 0)
+    (property "Reference" "C327" (id 0) (at 46.355 100.3299 0)
       (effects (font (size 1.27 1.27)) (justify left))
     )
@@
   (symbol (lib_id "Device:C") (at 114.935 122.555 0) (unit 1)
     (in_bom yes) (on_board yes) (fields_autoplaced)
-    (property "Reference" "C?" (id 0) (at 118.745 121.9199 0)
+    (property "Reference" "C328" (id 0) (at 118.745 121.9199 0)
       (effects (font (size 1.27 1.27)) (justify left))
     )
@@
   (symbol (lib_id "Device:C") (at 126.365 122.555 180) (unit 1)
     (in_bom yes) (on_board yes) (fields_autoplaced)
-    (property "Reference" "C?" (id 0) (at 130.175 121.9199 0)
+    (property "Reference" "C329" (id 0) (at 130.175 121.9199 0)
       (effects (font (size 1.27 1.27)) (justify right))
     )
@@
   (symbol (lib_id "Device:C") (at 214.63 193.04 0) (unit 1)
     (in_bom yes) (on_board yes) (fields_autoplaced)
-    (property "Reference" "C?" (id 0) (at 217.805 192.4049 0)
+    (property "Reference" "C330" (id 0) (at 217.805 192.4049 0)
       (effects (font (size 1.27 1.27)) (justify left))
     )
@@
   (symbol (lib_id "Switch:SW_Push") (at 33.655 101.6 90) (unit 1)
     (in_bom yes) (on_board yes) (fields_autoplaced)
-    (property "Reference" "SW?" (id 0) (at 34.925 100.9649 90)
+    (property "Reference" "SW301" (id 0) (at 34.925 100.9649 90)
       (effects (font (size 1.27 1.27)) (justify right))
     )
@@
   (symbol (lib_id "Device:FerriteBead") (at 132.08 116.84 90) (unit 1)
     (in_bom yes) (on_board yes) (fields_autoplaced)
-    (property "Reference" "FB?" (id 0) (at 132.08 110.49 90))
+    (property "Reference" "FB301" (id 0) (at 132.08 110.49 90))
     (property "Value" "FerriteBead" (id 1) (at 132.08 113.03 90)
       (effects (font (size 1.27 1.27)) hide)
@@
   (symbol (lib_id "Connector_Generic:Conn_01x05") (at 255.905 191.135 0) (unit 1)
     (in_bom yes) (on_board yes)
-    (property "Reference" "J?" (id 0) (at 250.19 198.7549 0)
+    (property "Reference" "J305" (id 0) (at 250.19 198.7549 0)
       (effects (font (size 1.27 1.27)) (justify left))
     )
@@
   (symbol (lib_id "Connector_Generic:Conn_01x06") (at 252.73 330.2 0) (unit 1)
     (in_bom yes) (on_board yes)
-    (property "Reference" "J?" (id 0) (at 255.27 330.8349 0)
+    (property "Reference" "J304" (id 0) (at 255.27 330.8349 0)
       (effects (font (size 1.27 1.27)) (justify left))
     )
@@
   (symbol (lib_id "Connector_Generic:Conn_02x05_Odd_Even") (at 242.57 301.625 0) (unit 1)
     (in_bom yes) (on_board yes)
-    (property "Reference" "J?" (id 0) (at 243.84 293.37 0))
+    (property "Reference" "J302" (id 0) (at 243.84 293.37 0))
     (property "Value" "FTSH-105-01-F-DV-007-K" (id 1) (at 243.84 294.005 0)
       (effects (font (size 1.27 1.27)) hide)
@@
   (symbol (lib_id "Connector:USB_B") (at 252.73 165.1 0) (mirror y) (unit 1)
     (in_bom yes) (on_board yes)
-    (property "Reference" "J?" (id 0) (at 251.46 155.7019 0)
+    (property "Reference" "J303" (id 0) (at 251.46 155.7019 0)
       (effects (font (size 1.27 1.27)) (justify right))
     )
@@
   (symbol (lib_id "Power_Protection:USBLC6-2SC6") (at 212.725 168.275 0) (unit 1)
     (in_bom yes) (on_board yes)
-    (property "Reference" "U?" (id 0) (at 207.01 159.385 0))
+    (property "Reference" "U303" (id 0) (at 207.01 159.385 0))
     (property "Value" "USBLC6-2SC6" (id 1) (at 203.835 177.8 0))
     (property "Footprint" "Package_TO_SOT_SMD:SOT-23-6" (id 2) (at 212.725 180.975 0)
